File: bubble size sensor.sch (EAGLE design)
At the start: 42 parts, among them P5 TPPAD1-13, P6 TPPAD1-13, P7 TPPAD1-13, U1 PINHD-1X6

Commit message: Schematic updated with new EEPROMs
Board layout still in progress.
Parts:
- removed IC1: (no value), ic-package:DIL8
- removed U$13, U$15: M2_SCREW_HOLE, kyle:M2_SCREW_HOLE
- removed U$17, U$18, U$19, U$20: UBOLT_HOLE, kyle:UBOLT_HOLE
- added C3: (no value), rcl:C-USC0603
- added H$13, H$15: M2_SCREW_HOLE, kyle:M2_SCREW_HOLE
- added H$17, H$18, H$19, H$20: UBOLT_HOLE, kyle:UBOLT_HOLE
- added U2, U3: M24M02-DR-1, Schuyler:M24M02-DR-1
Connections:
- net A4: now also U2.SDA, U3.SDA; no longer IC1.5
- net A5: now also U2.SCL, U3.SCL; no longer IC1.6
- net GND: now also C3.2, U2.!WC, U2.E2, U2.VSS, U3.!WC, U3.VSS; no longer IC1.1, IC1.2, IC1.4, IC1.7
- net VCC: now also C3.1, U2.VCC, U3.E2, U3.VCC; no longer IC1.3, IC1.8
Other:
- note added: "Arduino Pro Mini and LED/Photodiodes"
- note added: "Buoy Connectors"
- note added: "EEPROMs"
- note added: "Pin A4: SDA Pin A5: SCL"
- note added: "U-Bolt Holes and Screw Holes"
- moved on the sheet: A0, A1, A2, C1, JP1, PWR, R1, R4, R5, R6, U$1, U$11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
